File: light.sch (KiCad schematic (older format))
At the start: 0 parts

Commit message: Schematic & footprint should be done.
Parts:
- added BT1: Battery, Pin_Headers:Pin_Header_Straight_1x02_Pitch1.27mm, symbol Battery
- added C1, C2: 100 nF, Capacitors_THT:C_Disc_D5.0mm_W2.5mm_P5.00mm, symbol C
- added C3: 10 µF, Capacitors_THT:CP_Radial_Tantal_D5.0mm_P5.00mm, symbol CP
- added P1: CONN_01X02, Pin_Headers:Pin_Header_Straight_1x02_Pitch1.27mm, symbol CONN_01X02
- added U1: TSL252, Pin_Headers:Pin_Header_Straight_1x03_Pitch2.00mm, symbol TSL25x
- added U2: LF50CV-DG, TO_SOT_Packages_THT:TO-220-3_Horizontal, symbol LF50CDT-TR
Connections:
- new net: P1.1 (P1), U1.3 (OUT)
- new net +5V: C2.1, C3.1, U1.2 (Vdd), U2.3 (Vout)
- new net +BATT: BT1.1 (+), C1.1, U2.1 (Vin)
- new net GND: BT1.2 (-), C1.2, C2.2, C3.2, P1.2 (P2), U1.1 (GND), U2.2 (GND)
Changed lines of the file:
@@
 LIBS:contrib
 LIBS:valves
+LIBS:sensors
+LIBS:light-cache
 EELAYER 25 0
 EELAYER END
@@
 Sheet 1 1
 Title "Light Flicker Sensor"
-Date ""
+Date "2017-10-08"
 Rev "0"
 Comp ""
@@
 Comment4 ""
 $EndDescr
+$Comp
+L LF50CDT-TR U2
+U 1 1 59DA54F7
+P 5350 2750
+F 0 "U2" H 5050 3100 50  0000 L CNN
+F 1 "LF50CV-DG" H 5050 3000 50  0000 L CNN
+F 2 "TO_SOT_Packages_THT:TO-220-3_Horizontal" H 5350 2600 50  0001 L CNN
+F 3 "" H 5350 2900 50  0001 C CNN
+	1    5350 2750
+	1    0    0    -1
+$EndComp
+$Comp
+L C C1
+U 1 1 59DA558F
+P 4750 2900
+F 0 "C1" H 4775 3000 50  0000 L CNN
+F 1 "100 nF" H 4775 2800 50  0000 L CNN
+F 2 "Capacitors_THT:C_Disc_D5.0mm_W2.5mm_P5.00mm" H 4788 2750 50  0001 C CNN
+F 3 "" H 4750 2900 50  0000 C CNN
+F 4 "K104Z15Y5VE5TH5" H 4750 2900 60  0001 C CNN "P/N"
+	1    4750 2900
+	1    0    0    -1
+$EndComp
+$Comp
+L C C2
+U 1 1 59DA5760
+P 5850 2900
+F 0 "C2" H 5875 3000 50  0000 L CNN
+F 1 "100 nF" H 5875 2800 50  0000 L CNN
+F 2 "Capacitors_THT:C_Disc_D5.0mm_W2.5mm_P5.00mm" H 5888 2750 50  0001 C CNN
+F 3 "" H 5850 2900 50  0000 C CNN
+F 4 "K104Z15Y5VE5TH5" H 5850 2900 60  0001 C CNN "P/N"
+	1    5850 2900
+	1    0    0    -1
+$EndComp
+$Comp
+L CP C3
+U 1 1 59DA57AD
+P 6200 2900
+F 0 "C3" H 6225 3000 50  0000 L CNN
+F 1 "10 µF" H 6225 2800 50  0000 L CNN
+F 2 "Capacitors_THT:CP_Radial_Tantal_D5.0mm_P5.00mm" H 6238 2750 50  0001 C CNN
+F 3 "" H 6200 2900 50  0000 C CNN
+F 4 "TAP106K010CCS" H 6200 2900 60  0001 C CNN "P/N"
+	1    6200 2900
+	1    0    0    -1
+$EndComp
+$Comp
+L GND #PWR01
+U 1 1 59DA5897
+P 5950 3100
+F 0 "#PWR01" H 5950 2850 50  0001 C CNN
+F 1 "GND" H 5950 2950 50  0000 C CNN
+F 2 "" H 5950 3100 50  0000 C CNN
+F 3 "" H 5950 3100 50  0000 C CNN
+	1    5950 3100
+	1    0    0    -1
+$EndComp
+Wire Wire Line
+	4200 3100 7450 3100
+Wire Wire Line
+	4750 3100 4750 3050
+Wire Wire Line
+	5350 2950 5350 3100
+Connection ~ 5350 3100
+Wire Wire Line
+	5850 3050 5850 3100
+Connection ~ 5850 3100
+Wire Wire Line
+	6200 3100 6200 3050
+Connection ~ 5950 3100
+$Comp
+L TSL25x U1
+U 1 1 59DA5A95
+P 6900 2800
+F 0 "U1" H 6900 2550 60  0000 C TNN
+F 1 "TSL252" H 6900 3050 60  0000 C BNN
+F 2 "Pin_Headers:Pin_Header_Straight_1x03_Pitch2.00mm" H 6900 2400 60  0001 C CNN
+F 3 "" H 6900 2550 60  0001 C CNN
+	1    6900 2800
+	1    0    0    -1
+$EndComp
+Wire Wire Line
+	5750 2650 6500 2650
+Wire Wire Line
+	6500 2650 6500 2700
+$Comp
+L +5V #PWR02
+U 1 1 59DA5B1D
+P 6050 2500
+F 0 "#PWR02" H 6050 2350 50  0001 C CNN
+F 1 "+5V" H 6050 2640 50  0000 C CNN
+F 2 "" H 6050 2500 50  0000 C CNN
+F 3 "" H 6050 2500 50  0000 C CNN
+	1    6050 2500
+	1    0    0    -1
+$EndComp
+Wire Wire Line
+	6050 2500 6050 2650
+Connection ~ 6050 2650
+Wire Wire Line
+	6200 2750 6200 2650
+Connection ~ 6200 2650
+Wire Wire Line
+	5850 2750 5850 2650
+Connection ~ 5850 2650
+Wire Wire Line
+	4750 2750 4750 2650
+Wire Wire Line
+	4200 2650 4950 2650
+Wire Wire Line
+	6500 3100 6500 2900
+Connection ~ 6200 3100
+Wire Wire Line
+	6500 2800 6400 2800
+Wire Wire Line
+	6400 2800 6400 2300
+Wire Wire Line
+	6400 2300 7450 2300
+$Comp
+L CONN_01X02 P1
+U 1 1 59DA5C1A
+P 7650 2800
+F 0 "P1" H 7650 2950 50  0000 C CNN
+F 1 "CONN_01X02" V 7750 2800 50  0000 C CNN
+F 2 "Pin_Headers:Pin_Header_Straight_1x02_Pitch1.27mm" H 7650 2800 50  0001 C CNN
+F 3 "" H 7650 2800 50  0000 C CNN
+	1    7650 2800
+	1    0    0    -1
+$EndComp
+Wire Wire Line
+	7450 3100 7450 2850
+Connection ~ 6500 3100
+Wire Wire Line
+	7450 2300 7450 2750
+Connection ~ 4750 3100
+Connection ~ 4750 2650
+$Comp
+L +BATT #PWR03
+U 1 1 59DA5DD0
+P 4650 2550
+F 0 "#PWR03" H 4650 2400 50  0001 C CNN
+F 1 "+BATT" H 4650 2690 50  0000 C CNN
+F 2 "" H 4650 2550 50  0000 C CNN
+F 3 "" H 4650 2550 50  0000 C CNN
+	1    4650 2550
+	1    0    0    -1
+$EndComp
+Wire Wire Line
+	4650 2550 4650 2650
+Connection ~ 4650 2650
+$Comp
+L Battery BT1
+U 1 1 59DA5E15
+P 4200 2900
+F 0 "BT1" H 4300 3000 50  0000 L CNN
+F 1 "Battery" H 4300 2900 50  0000 L CNN
+F 2 "Pin_Headers:Pin_Header_Straight_1x02_Pitch1.27mm" V 4200 2960 50  0001 C CNN
+F 3 "" V 4200 2960 50  0000 C CNN
+	1    4200 2900
+	1    0    0    -1
+$EndComp
+Wire Wire Line
+	4200 2700 4200 2650
 $EndSCHEMATC

Commit message: Change some footprints and the regulator.
Parts:
- BT1, P1: footprint Pin_Headers:Pin_Header_Straight_1x02_Pitch1.27mm -> Connectors_Terminal_Blocks:TerminalBlock_bornier-2_P5.08mm
- U2: value LF50CV-DG -> LM340LAZ-5.0/NOPB; footprint TO_SOT_Packages_THT:TO-220-3_Horizontal -> Customs:TO-92_Inline_Narrow_Flip; Alternate 1 (none) -> L4931CZ50-AP; Alternate 2 (none) -> LM78L05ACZ/LFT1; Alternate 3 (none) -> LE50ABZ-AP; Alternates Note (none) -> Alternates footprints differ
Changed lines of the file:
@@
 Sheet 1 1
 Title "Light Flicker Sensor"
-Date "2017-10-08"
-Rev "0"
+Date ""
+Rev "1"
 Comp ""
 Comment1 ""
@@
 Comment4 ""
 $EndDescr
-$Comp
-L LF50CDT-TR U2
-U 1 1 59DA54F7
-P 5350 2750
-F 0 "U2" H 5050 3100 50  0000 L CNN
-F 1 "LF50CV-DG" H 5050 3000 50  0000 L CNN
-F 2 "TO_SOT_Packages_THT:TO-220-3_Horizontal" H 5350 2600 50  0001 L CNN
-F 3 "" H 5350 2900 50  0001 C CNN
-	1    5350 2750
-	1    0    0    -1
-$EndComp
 $Comp
 L C C1
@@
 	1    0    0    -1
 $EndComp
+$Comp
+L TSL25x U1
+U 1 1 59DA5A95
+P 6900 2800
+F 0 "U1" H 6900 2550 60  0000 C TNN
+F 1 "TSL252" H 6900 3050 60  0000 C BNN
+F 2 "Pin_Headers:Pin_Header_Straight_1x03_Pitch2.00mm" H 6900 2400 60  0001 C CNN
+F 3 "" H 6900 2550 60  0001 C CNN
+	1    6900 2800
+	1    0    0    -1
+$EndComp
+$Comp
+L +5V #PWR02
+U 1 1 59DA5B1D
+P 6050 2500
+F 0 "#PWR02" H 6050 2350 50  0001 C CNN
+F 1 "+5V" H 6050 2640 50  0000 C CNN
+F 2 "" H 6050 2500 50  0000 C CNN
+F 3 "" H 6050 2500 50  0000 C CNN
+	1    6050 2500
+	1    0    0    -1
+$EndComp
+$Comp
+L CONN_01X02 P1
+U 1 1 59DA5C1A
+P 7650 2800
+F 0 "P1" H 7650 2950 50  0000 C CNN
+F 1 "CONN_01X02" V 7750 2800 50  0000 C CNN
+F 2 "Connectors_Terminal_Blocks:TerminalBlock_bornier-2_P5.08mm" H 7650 2800 50  0001 C CNN
+F 3 "" H 7650 2800 50  0000 C CNN
+	1    7650 2800
+	1    0    0    -1
+$EndComp
+$Comp
+L +BATT #PWR03
+U 1 1 59DA5DD0
+P 4650 2550
+F 0 "#PWR03" H 4650 2400 50  0001 C CNN
+F 1 "+BATT" H 4650 2690 50  0000 C CNN
+F 2 "" H 4650 2550 50  0000 C CNN
+F 3 "" H 4650 2550 50  0000 C CNN
+	1    4650 2550
+	1    0    0    -1
+$EndComp
+$Comp
+L Battery BT1
+U 1 1 59DA5E15
+P 4200 2900
+F 0 "BT1" H 4300 3000 50  0000 L CNN
+F 1 "Battery" H 4300 2900 50  0000 L CNN
+F 2 "Connectors_Terminal_Blocks:TerminalBlock_bornier-2_P5.08mm" V 4200 2960 50  0001 C CNN
+F 3 "" V 4200 2960 50  0000 C CNN
+	1    4200 2900
+	1    0    0    -1
+$EndComp
 Wire Wire Line
 	4200 3100 7450 3100
@@
 	6200 3100 6200 3050
 Connection ~ 5950 3100
-$Comp
-L TSL25x U1
-U 1 1 59DA5A95
-P 6900 2800
-F 0 "U1" H 6900 2550 60  0000 C TNN
-F 1 "TSL252" H 6900 3050 60  0000 C BNN
-F 2 "Pin_Headers:Pin_Header_Straight_1x03_Pitch2.00mm" H 6900 2400 60  0001 C CNN
-F 3 "" H 6900 2550 60  0001 C CNN
-	1    6900 2800
-	1    0    0    -1
-$EndComp
 Wire Wire Line
 	5750 2650 6500 2650
 Wire Wire Line
 	6500 2650 6500 2700
-$Comp
-L +5V #PWR02
-U 1 1 59DA5B1D
-P 6050 2500
-F 0 "#PWR02" H 6050 2350 50  0001 C CNN
-F 1 "+5V" H 6050 2640 50  0000 C CNN
-F 2 "" H 6050 2500 50  0000 C CNN
-F 3 "" H 6050 2500 50  0000 C CNN
-	1    6050 2500
-	1    0    0    -1
-$EndComp
 Wire Wire Line
 	6050 2500 6050 2650
@@
 Wire Wire Line
 	6400 2300 7450 2300
-$Comp
-L CONN_01X02 P1
-U 1 1 59DA5C1A
-P 7650 2800
-F 0 "P1" H 7650 2950 50  0000 C CNN
-F 1 "CONN_01X02" V 7750 2800 50  0000 C CNN
-F 2 "Pin_Headers:Pin_Header_Straight_1x02_Pitch1.27mm" H 7650 2800 50  0001 C CNN
-F 3 "" H 7650 2800 50  0000 C CNN
-	1    7650 2800
-	1    0    0    -1
-$EndComp
 Wire Wire Line
 	7450 3100 7450 2850
@@
 Connection ~ 4750 3100
 Connection ~ 4750 2650
-$Comp
-L +BATT #PWR03
-U 1 1 59DA5DD0
-P 4650 2550
-F 0 "#PWR03" H 4650 2400 50  0001 C CNN
-F 1 "+BATT" H 4650 2690 50  0000 C CNN
-F 2 "" H 4650 2550 50  0000 C CNN
-F 3 "" H 4650 2550 50  0000 C CNN
-	1    4650 2550
-	1    0    0    -1
-$EndComp
 Wire Wire Line
 	4650 2550 4650 2650
 Connection ~ 4650 2650
+Wire Wire Line
+	4200 2700 4200 2650
 $Comp
-L Battery BT1
-U 1 1 59DA5E15
-P 4200 2900
-F 0 "BT1" H 4300 3000 50  0000 L CNN
-F 1 "Battery" H 4300 2900 50  0000 L CNN
-F 2 "Pin_Headers:Pin_Header_Straight_1x02_Pitch1.27mm" V 4200 2960 50  0001 C CNN
-F 3 "" V 4200 2960 50  0000 C CNN
-	1    4200 2900
+L LF50CDT-TR U2
+U 1 1 59DA54F7
+P 5350 2750
+F 0 "U2" H 5050 3100 50  0000 L CNN
+F 1 "LM340LAZ-5.0/NOPB" H 5050 3000 50  0000 L CNN
+F 2 "Customs:TO-92_Inline_Narrow_Flip" H 5350 2600 50  0001 L CNN
+F 3 "" H 5350 2900 50  0001 C CNN
+F 4 "L4931CZ50-AP" H 5350 2750 60  0001 C CNN "Alternate 1"
+F 5 "LM78L05ACZ/LFT1" H 5350 2750 60  0001 C CNN "Alternate 2"
+F 6 "LE50ABZ-AP" H 5350 2750 60  0001 C CNN "Alternate 3"
+F 7 "Alternates footprints differ" H 5350 2750 60  0001 C CNN "Alternates Note"
+	1    5350 2750
 	1    0    0    -1
 $EndComp
-Wire Wire Line
-	4200 2700 4200 2650
 $EndSCHEMATC
